File: Deckelplatine.brd (EAGLE design)
At the start: 110 x 75 mm, 74 parts, among them IC1 MAX1487EESA+, IC2 74HCT595D, IC3 74HCT595D, IC4 74HCT595D, IC5 74HCT595D, IC6 74HCT595D, J1 52808-2570, U1 LM2676S, X1 236-406/000-023, X2 233-502

Commit message: Vergessener Commit zur Version 1.0.1
Changed lines of the file:
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@@
 <attribute name="DESCRIPTION" value="Drill Drawing"/>
 <attribute name="PROJEKTNAME" value="xMZ-Mod-Touch-Deckelplatine"/>
-<attribute name="VERSION" value="0.9.5"/>
+<attribute name="VERSION" value="1.0.0"/>
 </attributes>
 <variantdefs>
@@
 <attribute name="VALUE" x="43.2156" y="19.169" size="1.27" layer="27" ratio="10" rot="R180"/>
 <attribute name="NAME" x="40.319" y="16.9986" size="1.27" layer="25" ratio="10" rot="R270"/>
+<attribute name="OC_FARNELL_ALTERNATIVE" value="8452210" x="41.1836" y="15.232" size="1.778" layer="27" rot="R90" display="off"/>
 </element>
 <element name="IC2" library="RA-GAS Projekte LTD" package="SO16" value="74HCT595D" x="78.5" y="57" smashed="yes" rot="R180">
@@
 <attribute name="MF" value="TAIWAN SEMICONDUCTOR" x="50.8" y="70.461" size="1.778" layer="27" rot="R90" display="off"/>
 <attribute name="MPN" value="LL4005G" x="50.8" y="70.461" size="1.778" layer="27" rot="R90" display="off"/>
-<attribute name="NAME" x="49.376" y="70.198" size="0.8128" layer="25" rot="R90"/>
+<attribute name="NAME" x="48.541" y="71.661" size="0.8128" layer="25" rot="R270"/>
 <attribute name="VALUE" x="53.794" y="67.798" size="1.27" layer="27" rot="R90"/>
 </element>
@@
 </element>
 <element name="F1" library="fuse-littlefuse" package="01110005MR" value="2AT" x="36.8092" y="69.99" smashed="yes">
-<attribute name="OC_FARNELL" value="1155771" x="36.8092" y="69.99" size="1.778" layer="27" display="off"/>
+<attribute name="OC_FARNELL" value="2413914" x="36.8092" y="69.99" size="1.778" layer="27" display="off"/>
 <attribute name="OC_FARNELL_ALTERNATIVE" value="01110005MR" x="36.8092" y="69.99" size="1.778" layer="27" display="off"/>
 <attribute name="MF" value="LITTELFUSE" x="36.8092" y="69.99" size="1.778" layer="27" display="off"/>
@@
 <attribute name="MPN" value="01110005MR" x="36.83" y="62.23" size="1.778" layer="27" font="vector" ratio="15" display="off"/>
 <attribute name="MF" value="LITTELFUSE" x="36.83" y="62.23" size="1.778" layer="27" font="vector" ratio="15" display="off"/>
-<attribute name="OC_FARNELL" value="1155771" x="36.83" y="62.23" size="1.778" layer="27" font="vector" ratio="15" display="off"/>
+<attribute name="OC_FARNELL" value="2413914" x="36.83" y="62.23" size="1.778" layer="27" font="vector" ratio="15" display="off"/>
 <attribute name="NAME" x="35.52" y="61.405" size="1.778" layer="25" ratio="10"/>
 <attribute name="VALUE" x="32.52" y="57.15" size="1.778" layer="27" ratio="10"/>
 </element>
-<element name="D1" library="diode" package="MELF-MLL41" value="LL4005G" x="54.483" y="56.769" rot="R270">
+<element name="D1" library="diode" package="MELF-MLL41" value="LL4005G" x="54.483" y="56.769" smashed="yes" rot="R270">
 <attribute name="MPN" value="LL4005G" x="54.483" y="56.769" size="1.778" layer="27" font="vector" ratio="15" rot="R270" display="off"/>
 <attribute name="MF" value="TAIWAN SEMICONDUCTOR" x="54.483" y="56.769" size="1.778" layer="27" font="vector" ratio="15" rot="R270" display="off"/>
 <attribute name="OC_FARNELL" value="1625106" x="54.483" y="56.769" size="1.778" layer="27" font="vector" ratio="15" rot="R270" display="off"/>
+<attribute name="NAME" x="52.143" y="57.273" size="0.8128" layer="25" rot="R270"/>
+<attribute name="VALUE" x="51.489" y="59.432" size="1.27" layer="27" rot="R270"/>
 </element>
 <element name="R1" library="RA-GAS Projekte LTD" package="R0603" value="10k" x="61.214" y="9.906" rot="R180">
@@
 <attribute name="MF" value="TAIWAN SEMICONDUCTOR" x="50.8" y="61.849" size="1.778" layer="27" font="vector" ratio="15" rot="R270" display="off"/>
 <attribute name="OC_FARNELL" value="1625106" x="50.8" y="61.849" size="1.778" layer="27" font="vector" ratio="15" rot="R270" display="off"/>
-<attribute name="NAME" x="52.624" y="62.712" size="0.8128" layer="25" rot="R270"/>
+<attribute name="NAME" x="48.56" y="62.585" size="0.8128" layer="25" rot="R270"/>
 <attribute name="VALUE" x="47.806" y="64.512" size="1.27" layer="27" rot="R270"/>
 </element>
@@
 <contactref element="L1" pad="1"/>
 <contactref element="D2" pad="C"/>
-<wire x1="36.13" y1="42.31" x2="40.64" y2="42.31" width="0.254" layer="1"/>
+<wire x1="36.13" y1="42.31" x2="40.64" y2="42.31" width="0.8128" layer="1"/>
 <wire x1="40.64" y1="42.31" x2="41.0953" y2="42.31" width="0.254" layer="1"/>
 <wire x1="41.0953" y1="42.31" x2="41.1153" y2="42.33" width="0.254" layer="1"/>
-<wire x1="38.24" y1="33.81" x2="38.24" y2="34.43" width="0.254" layer="1"/>
-<wire x1="38.24" y1="34.43" x2="40.64" y2="36.83" width="0.254" layer="1"/>
-<wire x1="40.64" y1="36.83" x2="40.64" y2="38.0417" width="0.254" layer="1"/>
-<wire x1="40.64" y1="38.0417" x2="41.0983" y2="38.5" width="0.254" layer="1"/>
-<wire x1="41.0983" y1="38.5" x2="41.0983" y2="41.8517" width="0.254" layer="1"/>
+<wire x1="38.24" y1="33.81" x2="38.24" y2="34.43" width="0.8128" layer="1"/>
+<wire x1="38.24" y1="34.43" x2="40.64" y2="36.83" width="0.8128" layer="1"/>
+<wire x1="40.64" y1="36.83" x2="40.64" y2="38.0417" width="0.8128" layer="1"/>
+<wire x1="40.64" y1="38.0417" x2="41.0983" y2="38.5" width="0.8128" layer="1"/>
+<wire x1="41.0983" y1="38.5" x2="41.0983" y2="41.8517" width="0.8128" layer="1"/>
 <wire x1="41.0983" y1="41.8517" x2="40.64" y2="42.31" width="0.254" layer="1"/>
 </signal>
